File: PCB/USB_Geocache.kicad_pcb (KiCad board)
At the start: 4 copper layers, 25.5 x 49 mm, 47 parts, among them P1 USB_Mini_B, P2 Battery, P3 SWD, P4 GPS, P5 Button, P7 Servo, Q1 SI2301BDS-T1-E3, Q2 BST82, Q3 SI2301BDS-T1-E3, U1 MCP73831/OT, U2 ILI9341_LCD_Breakout, U3 LPC11U24FBD48, U4 LM3670MF, U5 25LC640A-I/SN, X1 12.000MHz

Commit message: Updated schematics for STM32F072
* No crystal required for USB
* Higher SPI speed (18MHz)
* Simplified some circuits
* Fixed current draw issues (e.g. for Vmeas resistor divider)
Parts:
- removed JP1: Jumper_NO_Small, Capacitors_SMD:C_0805
- removed P1: USB_Mini_B, Connect:USB_Mini-B
- removed X1: 12.000MHz, Components:crystal_SMD_5032
- added C15: C, Capacitor_SMD:C_0805_2012Metric, B.Cu at (208.0, -47.5)
- added J1: USB_B_Mini, Connector_USB:USB_Mini-B_Lumber_2486_Horizontal, F.Cu at (119.5, -50.0)
- added Q4: DMP3099L, Package_TO_SOT_SMD:SOT-23_Handsoldering, F.Cu at (240.5, -1.50)
- added R14: 4K7, Resistor_SMD:R_0805_2012Metric, F.Cu at (239.5, -6.00)
- added R15: 4K7, Resistor_SMD:R_0805_2012Metric, F.Cu at (236.0, -0.50)
- added R16: 10K, Resistor_SMD:R_0805_2012Metric, F.Cu at (235.5, -7.00)
- added R17: R, Resistor_SMD:R_0805_2012Metric, F.Cu at (119.5, -43.5)
- added R18: R, Resistor_SMD:R_0805_2012Metric, F.Cu at (121.5, -43.5)
- added R19: R, Resistor_SMD:R_0805_2012Metric, F.Cu at (117.5, -43.5)
- C1, C10, C12, C14, C2: footprint Capacitors_SMD:C_0805_HandSoldering -> Capacitor_SMD:C_0805_2012Metric; moved to F.Cu
- C11: value 18pF -> C; footprint Capacitors_SMD:C_0805_HandSoldering -> Capacitor_SMD:C_0805_2012Metric
- C13, C16, C3, C4, C8: footprint Capacitors_SMD:C_0805_HandSoldering -> Capacitor_SMD:C_0805_2012Metric
- C5: value 10uF -> 0.1uF; footprint Capacitors_SMD:C_0805_HandSoldering -> Capacitor_SMD:C_0805_2012Metric
- C6: value 18pF -> C; footprint Capacitors_SMD:C_0805_HandSoldering -> Capacitor_SMD:C_0805_2012Metric; moved to F.Cu
- C7, C9: value 0.1uF -> C; footprint Capacitors_SMD:C_0805_HandSoldering -> Capacitor_SMD:C_0805_2012Metric
- D2, D3: footprint Diodes_SMD:SOD-123 -> Diode_SMD:D_SOD-123; moved to F.Cu
- L1: footprint Resistors_SMD:R_1210_HandSoldering -> Inductor_SMD:L_Taiyo-Yuden_NR-24xx_HandSoldering
- P2: footprint Connectors_JST:JST_PH_S02B-PH-K-S_02x2.00mm_Angled -> Connector_JST:JST_PH_S2B-PH-K_1x02_P2.00mm_Horizontal
- P3: footprint Components:POGO_Connector -> Connector_PinHeader_1.27mm:PinHeader_1x06_P1.27mm_Vertical
- P4: footprint Connectors_JST:JST_PH_S04B-PH-K-S_04x2.00mm_Angled -> Connector_JST:JST_PH_S4B-PH-K_1x04_P2.00mm_Horizontal
- P5: footprint Pin_Headers:Pin_Header_Straight_1x02 -> Connector_PinHeader_2.54mm:PinHeader_1x02_P2.54mm_Vertical
- P7: footprint Pin_Headers:Pin_Header_Angled_1x03 -> Connector_PinHeader_2.54mm:PinHeader_1x03_P2.54mm_Horizontal
- Q1: value SI2301BDS-T1-E3 -> DMP3099L; footprint TO_SOT_Packages_SMD:SOT-23_Handsoldering -> Package_TO_SOT_SMD:SOT-23_Handsoldering; moved to F.Cu
- Q2: value BST82 -> DMP3099L; footprint TO_SOT_Packages_SMD:SOT-23_Handsoldering -> Package_TO_SOT_SMD:SOT-23_Handsoldering; moved to F.Cu
- Q3: value SI2301BDS-T1-E3 -> DMP3099L; footprint TO_SOT_Packages_SMD:SOT-23_Handsoldering -> Package_TO_SOT_SMD:SOT-23_Handsoldering
- R1, R11, R13, R3, R5, R6: footprint Resistors_SMD:R_0805_HandSoldering -> Resistor_SMD:R_0805_2012Metric; moved to F.Cu
- R10: value 4K7 -> 10K; footprint Resistors_SMD:R_0805_HandSoldering -> Resistor_SMD:R_0805_2012Metric; moved to F.Cu
- R12, R7, R8, R9: footprint Resistors_SMD:R_0805_HandSoldering -> Resistor_SMD:R_0805_2012Metric
- R2: value 4K7 -> 10K; footprint Resistors_SMD:R_0805_HandSoldering -> Resistor_SMD:R_0805_2012Metric
- R4: value 470 -> 10K; footprint Resistors_SMD:R_0805_HandSoldering -> Resistor_SMD:R_0805_2012Metric
- U1: value MCP73831/OT -> MCP73831-2-OT; footprint TO_SOT_Packages_SMD:SOT-23-5 -> Package_TO_SOT_SMD:TSOT-23-5_HandSoldering
- U2: value ILI9341_LCD_Breakout -> LM3670MF; footprint Pin_Headers:Pin_Header_Straight_1x09 -> Package_TO_SOT_SMD:TSOT-23-5_HandSoldering
- U3: value LPC11U24FBD48 -> STM32F072C8Tx; footprint QFP:LQFP-48_7x7mm_Pitch0.5mm -> Package_QFP:TQFP-48_7x7mm_P0.5mm
- U4: value LM3670MF -> CR2013-MI2120; footprint TO_SOT_Packages_SMD:SOT-23-5 -> Display:CR2013-MI2120
- U5: footprint SOIC_Packages:SOIC-8_3.9x4.9mm_Pitch1.27mm -> Package_SO:SOIC-8_3.9x4.9mm_P1.27mm; moved to F.Cu
- moved R1 178.0 mm to (273.0, -34.5), turned to 0 degrees
- moved P7 164.9 mm to (269.0, -26.0), turned to 0 degrees
- moved P2 164.2 mm to (255.5, -63.0), turned to 0 degrees
- moved Q1 164.1 mm to (264.5, -26.5), turned to 0 degrees
- moved R8 163.9 mm to (267.5, -31.0), turned to 0 degrees
- moved R12 147.9 mm to (262.5, -17.0), turned to 0 degrees
- moved R9 145.9 mm to (78.5, -15.0)
- moved R13 142.4 mm to (262.5, -20.5), turned to 0 degrees
- moved C14 140.6 mm to (267.5, -17.5), turned to 0 degrees
- moved C7 138.8 mm to (203.5, -47.0)
- moved Q3 137.6 mm to (79.0, -11.5)
- moved Q2 137.3 mm to (157.5, -44.0), turned to 0 degrees
- moved U3 136.2 mm to (206.0, -45.0)
- moved C16 135.8 mm to (276.5, 15.0), turned to 0 degrees
- moved C9 135.4 mm to (204.0, -42.5), turned to 0 degrees
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Connections:
- net /Rsense renamed Net-(P7-Pad3)
- net Net-(U3-Pad34) renamed /SWDIO
- C1 pad 1: +3V3 -> Net-(C1-Pad1)
- C11 pad 1: /XIN -> +3V3
- C12 pad 1: GND -> +3V3
- C12 pad 2: +3V3 -> GND
- C14 pad 1: /Vsense -> /I_SERVO
- C2 pad 1: +3V3 -> Net-(C1-Pad1)
- C5 pad 1: +3V3 -> /SW_RESET
- C6 pad 1: /XOUT -> /V_BATT
- D2 pad 2: /Button -> /BUTTON
- D3 pad 2: /Enable -> /SW_ENABLE
- L1 pad 1: Net-(L1-Pad1) -> +3V3
- L1 pad 2: +3V3 -> Net-(L1-Pad2)
- P3 pad 2: /SW_CLK -> /SW_DIO
- P3 pad 3: (no net) -> /SW_CLK
- P3 pad 4: Net-(P3-Pad4) -> /SW_RESET
- P3 pad 5: /SW_RESET -> Net-(P3-Pad5)
- P4 pad 1: +3V3 -> Net-(C1-Pad1)
- P4 pad 2: GND -> /GPS_RX
- P4 pad 3: /GPS_RX -> /GPS_TX
- P4 pad 4: /GPS_TX -> GND
- P5 pad 2: /Button -> /BUTTON
- P7 pad 1: /SERVO_SIGNAL -> /SERVO_PWM
- Q1 pad 1: Net-(Q1-Pad1) -> /SERVO_EN
- Q2 pad 1: /SERVO_EN -> /GPS_PWR
- Q2 pad 2: GND -> +3V3
- Q2 pad 3: Net-(Q1-Pad1) -> Net-(C1-Pad1)
- Q3 pad 1: /BL -> /LDC_BL
- R1 pad 1: Net-(Q1-Pad1) -> /SERVO_EN
- R10 pad 1: /Button -> /BUTTON
- R13 pad 1: /Vsense -> /I_SERVO
- R2 pad 2: Net-(JP1-Pad1) -> /GPS_RX
- R3 pad 2: /GPS_RX -> /GPS_PWR
- R4 pad 1: /BATT_STAT -> +3V3
- R4 pad 2: +5V -> /GPS_TX
- R5 pad 1: /SERVO_EN -> +3V3
- R5 pad 2: GND -> /SW_RESET
- R8 pad 2: /SERVO_SIGNAL -> /SERVO_PWM
- R9 pad 2: /BL -> /LDC_BL
- U1 pad 1: /BATT_STAT -> Net-(U1-Pad1)
- U2 pad 1: +3V3 -> +BATT
- U2 pad 3: /LCD_CS -> /EN
- U2 pad 4: /LCD_RESET -> +3V3
- U2 pad 5: /LCD_DC -> Net-(L1-Pad2)
- U3 pad 1: Net-(U3-Pad1) -> +3V3
- U3 pad 10: Net-(U3-Pad10) -> /V_BATT
- U3 pad 11: /GPS_RX -> /I_SERVO
- U3 pad 13: /SERVO_EN -> /GPS_RX
- U3 pad 14: +5V -> /GPS_PWR
- U3 pad 15: Net-(U3-Pad15) -> /SPI_SCK
- U3 pad 16: Net-(U3-Pad16) -> /SPI_MISO
- U3 pad 17: Net-(U3-Pad17) -> /SPI_MOSI
- U3 pad 18: Net-(U3-Pad18) -> /LCD_CS
- U3 pad 19: /D- -> /LCD_DC
- U3 pad 20: /D+ -> /LDC_BL
- U3 pad 21: /SERVO_SIGNAL -> Net-(U3-Pad21)
- U3 pad 23: /EEPROM_CS -> GND
- U3 pad 24: Net-(U3-Pad24) -> +3V3
- U3 pad 25: /BL -> Net-(U3-Pad25)
- U3 pad 26: Net-(U3-Pad26) -> /VMEAS_CTRL
- U3 pad 27: /SPI_MISO -> Net-(U3-Pad27)
- U3 pad 28: /SPI_MOSI -> Net-(U3-Pad28)
- U3 pad 29: /SW_CLK -> /SERVO_PWM
- U3 pad 3: /SW_RESET -> Net-(U3-Pad3)
- U3 pad 30: Net-(U3-Pad30) -> /SERVO_EN
- U3 pad 31: /SPI_SCK -> Net-(U3-Pad31)
- U3 pad 32: /Button -> /USB_D-
- U3 pad 33: /Vsense -> /USB_D+
- U3 pad 35: /LCD_DC -> GND
- U3 pad 36: /LCD_RESET -> +3V3
- U3 pad 37: /LCD_CS -> /SWCLK
- U3 pad 38: /Enable -> Net-(U3-Pad38)
- U3 pad 39: /SW_CLK -> /LCD_RESET
- U3 pad 4: Net-(JP1-Pad1) -> Net-(U3-Pad4)
- U3 pad 40: /BATT_STAT -> Net-(U3-Pad40)
- U3 pad 41: GND -> /CS_EEPROM
- U3 pad 44: +3V3 -> Net-(U3-Pad44)
- U3 pad 45: Net-(U3-Pad45) -> /BUTTON
- U3 pad 46: Net-(U3-Pad46) -> /SW_ENABLE
- U3 pad 47: Net-(U3-Pad47) -> GND
- U3 pad 48: Net-(U3-Pad48) -> +3V3
- U3 pad 5: GND -> Net-(U3-Pad5)
- U3 pad 6: /XIN -> Net-(U3-Pad6)
- U3 pad 7: /XOUT -> /SW_RESET
- U3 pad 8: +3V3 -> GND
- U3 pad 9: Net-(U3-Pad9) -> +3V3
- U4 pad 1: +BATT -> +3V3
- U4 pad 3: /EN -> /LCD_CS
- U4 pad 4: +3V3 -> /LCD_RESET
- U4 pad 5: Net-(L1-Pad1) -> /LCD_DC
- U5 pad 1: /EEPROM_CS -> /CS_EEPROM
Routing:
- net GND: track 167.3 -> 0.00 mm, vias 9 -> 0
- net +3V3: track 159.5 -> 0.00 mm, vias 6 -> 0
- net +BATT: track 82.4 -> 0.00 mm, vias 2 -> 0
- net +5V: track 60.8 -> 0.00 mm, vias 3 -> 0
- net /SW_CLK: track 39.0 -> 0.00 mm, vias 2 -> 0
- net /D+: track 32.8 -> 0.00 mm, vias 2 -> 0
- net /D-: track 32.3 -> 0.00 mm, vias 2 -> 0
- net /BL: track 31.5 -> 0.00 mm, vias 2 -> 0
- net /Button: track 28.2 -> 0.00 mm, vias 1 -> 0
- net /BATT_STAT: track 21.0 -> 0.00 mm, vias 2 -> 0
- net /SPI_MISO: track 19.7 -> 0.00 mm, vias 1 -> 0
- net /SPI_MOSI: track 16.5 -> 0.00 mm, vias 1 -> 0
- net Net-(P7-Pad3): track 16.0 -> 0.00 mm
- net /EN: track 15.8 -> 0.00 mm, vias 1 -> 0
- net /SERVO_SIGNAL: track 14.7 -> 0.00 mm
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- removed copper zone on PWR, net +3V3
- removed copper zone on B.Cu, net GND
- removed copper zone on F.Cu, net GND
- removed copper zone on GND, net GND
Other:
- board outline removed
- board text removed: "+"
- board text removed: "-"
- board text removed: "Battery"
- board text removed: "Button"
- board text removed: "GND V+ PWM"
- board text removed: "GPS"
- board text removed: "RX"
- board text removed: "Reverse Geocache rev C 04/16"
- board text removed: "Servo"
- board text removed: "USB"
- board text removed: "V+"
- board text removed: "V-"

Commit message: PCB Layout
- Completed PCB layout for new processor (Rev C)
Parts:
- added C17: 18pF, Capacitor_SMD:C_0805_2012Metric, F.Cu at (197.2, 87.5)
- added C18: 18pF, Capacitor_SMD:C_0805_2012Metric, F.Cu at (205.2, 87.5)
- added J2: USB_ALT, Connector_PinHeader_2.54mm:PinHeader_1x05_P2.54mm_Vertical, B.Cu at (205.5, 62.0)
- added JP1: Boot, Jumper:SolderJumper-2_P1.3mm_Open_RoundedPad1.0x1.5mm, B.Cu at (207.8, 83.8)
- added JP2: 5V, Jumper:SolderJumper-2_P1.3mm_Open_RoundedPad1.0x1.5mm, B.Cu at (193.5, 68.0)
- added R20: 10K, Resistor_SMD:R_0805_2012Metric, B.Cu at (208.8, 81.2)
- added Y1: 8MHz, Crystal:Crystal_SMD_5032-4Pin_5.0x3.2mm, F.Cu at (201.2, 87.5)
- C11, C15, C7, C9: moved to F.Cu
- C13, C16, C5, J1, L1, P2, P3, P4, P5, P7, R10, R5, R6, U2, U3: moved to B.Cu
- R12: footprint Resistor_SMD:R_0805_2012Metric -> Resistor_SMD:R_1210_3225Metric
- moved R2 155.4 mm to (191.5, 96.4)
- moved R4 155.3 mm to (189.0, 96.4)
- moved R9 150.0 mm to (188.0, 87.5), turned to 270 degrees
- moved P4 148.1 mm to (193.5, 92.8), turned to 180 degrees
- moved R1 147.4 mm to (203.5, 95.5), turned to 270 degrees
- moved P2 147.0 mm to (187.8, 67.5)
- moved C1 146.0 mm to (198.0, 90.8)
- moved Q2 145.6 mm to (196.5, 96.2), turned to 180 degrees
- moved C2 145.4 mm to (198.0, 92.8)
- moved R3 145.1 mm to (200.5, 96.2), turned to 270 degrees
- moved Q3 144.3 mm to (184.0, 87.5), turned to 180 degrees
- moved J1 142.0 mm to (199.2, 67.5), turned to 270 degrees
- moved R19 141.7 mm to (204.0, 68.8), turned to 0 degrees
- moved R17 138.9 mm to (204.0, 66.8), turned to 180 degrees
- moved R8 138.2 mm to (204.5, 92.0)
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Connections:
- P3 pad 2: /SW_DIO -> /SWDIO
- P3 pad 3: /SW_CLK -> /SWCLK
- P4 pad 2: /GPS_RX -> /GPS_TX
- P4 pad 3: /GPS_TX -> /GPS_RX
- R2 pad 2: /GPS_RX -> /GPS_TX
- R4 pad 2: /GPS_TX -> /GPS_RX
- U3 pad 10: /V_BATT -> /I_SERVO
- U3 pad 11: /I_SERVO -> /V_BATT
- U3 pad 18: /LCD_CS -> /LCD_DC
- U3 pad 19: /LCD_DC -> /LCD_RESET
- U3 pad 20: /LDC_BL -> /LCD_CS
- U3 pad 21: Net-(U3-Pad21) -> /CS_EEPROM
- U3 pad 22: Net-(U3-Pad22) -> /LDC_BL
- U3 pad 39: /LCD_RESET -> Net-(U3-Pad39)
- U3 pad 40: Net-(U3-Pad40) -> /SW_ENABLE
- U3 pad 41: /CS_EEPROM -> /BUTTON
- U3 pad 45: /BUTTON -> Net-(U3-Pad45)
- U3 pad 46: /SW_ENABLE -> Net-(U3-Pad46)
Routing:
- net GND: track 0.00 -> 118.3 mm, vias 0 -> 19
- net +BATT: track 0.00 -> 103.8 mm, vias 0 -> 3
- net +3V3: track 0.00 -> 61.7 mm, vias 0 -> 10
- net /SERVO_PWM: track 0.00 -> 29.9 mm, vias 0 -> 1
- net /SPI_MOSI: track 0.00 -> 29.9 mm, vias 0 -> 1
- net /V_BATT: track 0.00 -> 29.5 mm, vias 0 -> 3
- net /SPI_MISO: track 0.00 -> 29.1 mm, vias 0 -> 1
- net /EN: track 0.00 -> 29.0 mm, vias 0 -> 1
- net /SERVO_EN: track 0.00 -> 28.0 mm, vias 0 -> 2
- net Net-(J1-Pad4): track 0.00 -> 27.2 mm, vias 0 -> 1
- net +5V: track 0.00 -> 25.2 mm, vias 0 -> 1
- net /GPS_PWR: track 0.00 -> 24.9 mm, vias 0 -> 2
- net /LDC_BL: track 0.00 -> 23.0 mm, vias 0 -> 2
- net Net-(J1-Pad3): track 0.00 -> 22.5 mm, vias 0 -> 1
- net /SW_RESET: track 0.00 -> 21.2 mm, vias 0 -> 1
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- added copper zone on PWR, net +3V3
- added copper zone on B.Cu, net GND
- added copper zone on F.Cu, net GND
- added copper zone on GND, net GND
Other:
- board outline added: 40 x 40 mm
- net class Default: via_dia 1.143 -> 0.75; via_drill 0.635 -> 0.35
- net class TestNet removed
- rule via_min_drill: 0.508 -> 0.3
- rule via_min_size: 1.143 -> 0.6
- board text added: "+"
- board text added: "-"
- board text added: "Battery"
- board text added: "Button"
- board text added: "GND"
- board text added: "GPS"
- board text added: "PWM V+ GND"
- board text added: "RX TX 3.3V"
- board text added: "Reverse Geocache Rev C March 2018"
- board text added: "SERVO"
- board text added: "USB"

Commit message: Further PCB tweaks
Routing:
- net GND: track 118.3 -> 124.3 mm, vias 19 -> 20
- net +3V3: track 61.7 -> 63.9 mm, vias 10 -> 11
- net +BATT: track 103.8 -> 106.0 mm
- net Net-(J1-Pad2): track 14.8 -> 16.1 mm
- net Net-(J1-Pad3): track 22.5 -> 23.1 mm
